File: Pistol_Camera_Driver/Pistol_Camera_Driver.kicad_pcb (KiCad board)
At the start: 2 copper layers, 70 x 92.7 mm, 105 parts, among them J1 Screw_Terminal_01x02, J10 I2C, J11 Screw_Terminal_01x02, J12 Screw_Terminal_01x02, J13 I2C, J18 Screw_Terminal_01x02, J19 I2C, J2 Objective, J21 Conn_02x08_Odd_Even, J22 Conn_02x08_Odd_Even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

Commit message: some test
Parts:
- added J3: Screw_Terminal_01x02, Connector_JST:JST_XH_B2B-XH-A_1x02_P2.50mm_Vertical, F.Cu at (-22.0, -51.4)
- added J5: Screw_Terminal_01x02, Connector_JST:JST_XH_B2B-XH-A_1x02_P2.50mm_Vertical, B.Cu at (-101.9, -57.0)
- J2: moved to F.Cu
- moved J1 84.4 mm to (-100.8, -44.6)
- moved J10 84.4 mm to (-88.5, -63.8)
- moved J13 84.4 mm to (-62.5, -65.8)
- moved J19 84.4 mm to (-76.0, -65.8)
- moved J21 84.4 mm to (-40.0, -55.6)
- moved J4 84.4 mm to (-101.8, -38.5)
- moved J6 84.4 mm to (-46.5, -65.7)
- moved R21 84.4 mm to (-88.2, -67.8)
- moved R23 84.4 mm to (-88.2, -66.3)
- moved REF** 84.4 mm to (-101.2, -64.8)
- moved REF** 84.4 mm to (-39.2, -28.8)
- moved REF** 84.4 mm to (-39.2, -64.8)
- moved REF** 84.4 mm to (-101.2, -28.8)
- moved SW1 84.4 mm to (-91.0, -32.9)
- moved SW2 84.4 mm to (-82.4, -32.9)
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Routing:
- net VBUS: track 156.3 -> 171.2 mm
- net SW3: track 10.1 -> 16.6 mm
- net GND: track 27.0 -> 24.9 mm, vias 327 -> 332
Other:
- board size 70 x 92.7 mm -> 139.9 x 46.1 mm
