File: Pistol_Camera_Driver/Pistol_Camera_Driver.kicad_sch (KiCad schematic)
At the start: 98 parts, among them J1 Screw_Terminal_01x02, J10 I2C, J11 Screw_Terminal_01x02, J12 Screw_Terminal_01x02, J13 I2C, J18 Screw_Terminal_01x02, J19 I2C, J2 Objective, J21 Conn_02x08_Odd_Even, J22 Conn_02x08_Odd_Even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

Commit message: some test
Parts:
- added J3, J5: Screw_Terminal_01x02, Connector_JST:JST_XH_B2B-XH-A_1x02_P2.50mm_Vertical, symbol Connector:Screw_Terminal_01x02
Connections:
- net GND: now also J3.2 (Pin_2), J5.2 (Pin_2)
- net VBUS: now also J3.1 (Pin_1), J5.1 (Pin_1)
